Commit message: Package modified

File: description/4w_testbot.xacro (robot description, xacro)
@@ -20,5 +20,5 @@
   <xacro:macro name="box_inertia" params="m w h d">
     <inertial>
-      <origin xyz="0 0 0.05" rpy="0 0 0"/>
+      <origin xyz="0 0 0.0358" rpy="0 0 0"/>
       <mass value="${m}"/>
       <inertia ixx="${(m/12) * (h*h + d*d)}" ixy="0.0" ixz="0.0" iyy="${(m/12) * (w*w + d*d)}" iyz="0.0" izz="${(m/12) * (w*w + h*h)}"/>
@@ -48,10 +48,10 @@
       <origin xyz="0.0 0.0 0.05" rpy="0.0 0.0 0.0"/>
     </collision>
-    <xacro:box_inertia m="2.5" w="0.4" d="0.6" h="0.2"/>
+    <xacro:box_inertia m="3.5" w="0.4" d="0.6" h="0.2"/>
   </link>
   <joint name="base_body_footprint_joint" type="fixed">
     <parent link="base_footprint"/>
     <child link="base_link"/>
-    <origin xyz="0.0 0.0 0.1" rpy="0.0 0.0 0.0"/>
+    <origin xyz="0.0 0.0 0.15" rpy="0.0 0.0 0.0"/>
   </joint>
   <!-- LIDAR -->
@@ -131,5 +131,5 @@
         </surface>
       </collision>
-      <xacro:cylinder_inertia m="1.0" r="0.1" h="0.05"/>
+      <xacro:cylinder_inertia m="0.05" r="0.1" h="0.05"/>
     </link>
     <joint name="${name}_joint" type="continuous">
@@ -141,8 +141,8 @@
     </joint>
   </xacro:macro>
-  <xacro:wheel name="rr_wheel" xyz="-0.18 -0.233 0.0" rpy="1.57 0 0"/>
-  <xacro:wheel name="fr_wheel" xyz="0.18 -0.233 0.0" rpy="1.57 0 0"/>
-  <xacro:wheel name="fl_wheel" xyz="0.18 0.233 0.0" rpy="1.57 0 0"/>
-  <xacro:wheel name="rl_wheel" xyz="-0.18 0.233 0.0" rpy="1.57 0 0"/>
+  <xacro:wheel name="rr_wheel" xyz="-0.18 -0.233 -0.05" rpy="1.57 0 0"/>
+  <xacro:wheel name="fr_wheel" xyz="0.18 -0.233 -0.05" rpy="1.57 0 0"/>
+  <xacro:wheel name="fl_wheel" xyz="0.18 0.233 -0.05" rpy="1.57 0 0"/>
+  <xacro:wheel name="rl_wheel" xyz="-0.18 0.233 -0.05" rpy="1.57 0 0"/>
   <!-- IMU -->
   <link name="imu_link"/>
@@ -228,4 +228,5 @@
       <state_interface name="position"/>
       <state_interface name="velocity"/>
+      <state_interface name="effort"/>
     </joint>
     <joint name="rr_wheel_joint">
@@ -236,4 +237,5 @@
       <state_interface name="position"/>
       <state_interface name="velocity"/>
+      <state_interface name="effort"/>
     </joint>
     <joint name="fl_wheel_joint">
@@ -244,4 +246,5 @@
       <state_interface name="position"/>
       <state_interface name="velocity"/>
+      <state_interface name="effort"/>
     </joint>
     <joint name="rl_wheel_joint">
@@ -252,5 +255,18 @@
       <state_interface name="position"/>
       <state_interface name="velocity"/>
-    </joint>
+      <state_interface name="effort"/>
+    </joint>
+     <sensor name="imu_sensor">
+    <state_interface name="orientation.x"/>
+    <state_interface name="orientation.y"/>
+    <state_interface name="orientation.z"/>
+    <state_interface name="orientation.w"/>
+    <state_interface name="angular_velocity.x"/>
+    <state_interface name="angular_velocity.y"/>
+    <state_interface name="angular_velocity.z"/>
+    <state_interface name="linear_acceleration.x"/>
+    <state_interface name="linear_acceleration.y"/>
+    <state_interface name="linear_acceleration.z"/>
+  </sensor>
   </ros2_control>
   <gazebo>
